File: PCB_kicad/alpha_pro_micro.sch (KiCad schematic (older format))
At the start: 67 parts, among them J1 Conn_01x03, J2 Conn_01x01_Female, J3 Conn_01x01_Female, J4 Conn_01x01_Female, J5 Conn_01x01_Female, J6 Conn_01x01_Female, J7 Conn_01x01_Female, J8 Conn_01x01_Female, J9 Conn_01x01_Female, K1 KEYSW, K10 KEYSW, K11 KEYSW, K12 KEYSW, K13 KEYSW, K14 KEYSW, K15 KEYSW, K16 KEYSW, K17 KEYSW, K18 KEYSW, K19 KEYSW, K2 KEYSW, K20 KEYSW, K21 KEYSW, K22 KEYSW, K23 KEYSW, K24 KEYSW, K25 KEYSW, K26 KEYSW, K27 KEYSW, K28 KEYSW, K3 KEYSW, K4 KEYSW, K5 KEYSW, K6 KEYSW, K7 KEYSW, K8 KEYSW, K9 KEYSW, SW1 SW_Push, U1 ProMicro

Commit message: Swapped switch footprint
Swapped switch footprint over to MX only, with LED support, and added support for LED driver and rest button.
Parts:
- removed J2, J3, J4, J5, J6, J7, J8, J9: Conn_01x01_Female, Connector_PinHeader_2.54mm:PinHeader_1x01_P2.54mm_Vertical, symbol Connector:Conn_01x01_Female
- added Q1: SMD-MOSFET-N-CH-60V-300MA-LOGIC-LEVEL-FET-2N7002_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, OPL_Discrete_Semiconductor:SOT-23, symbol OPL_Discrete_Semiconductor:SMD-MOSFET-N-CH-60V-300MA-LOGIC-LEVEL-FET-2N7002_SOT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
- added R1, R10, R11, R12, R13, R14, R15, R16, R17, R18, R19, R2, R20, R21, R22, R23, R24, R25, R26, R27, R28, R3, R4, R5, R6, R7, R8, R9: SMD-RES-4.7K-5%-1_8W_0805_, OPL_Resistor:PR-D1.8_L3.3MM, symbol OPL_Resistor:SMD-RES-4.7K-5%-1_8W_0805_
- added R29: SMD-RES-100K-5%-1_8W_0805_, OPL_Resistor:PR-D1.8_L3.3MM, symbol OPL_Resistor:SMD-RES-4.7K-5%-1_8W_0805_
- K1, K10, K11, K12, K13, K14, K15, K16, K17, K18, K19, K2, K20, K21, K22, K23, K24, K26, K27, K28, K3, K4, K5, K6, K7, K8, K9: footprint keebio-parts:MX-Alps-Choc-1U-NoLED -> MX_Alps_Hybrid:MXOnly-1U; symbol alpha_pro_micro-rescue:KEYSW -> keebio:MX-with-LED
- K25: symbol alpha_pro_micro-rescue:KEYSW -> keebio:MX-with-LED
Connections:
- net labels added: LED, LED_Out
- wire segments 202 -> 330
Other:
- moved on the sheet: D21, D22, D23, D24, D25, D26, D27, D28
